Commit message: some inertia problems fixed and files were edited.

File: src/pavlov_description/urdf/pavlov_mini.urdf.xacro (robot description, xacro)
@@ -236,5 +236,5 @@
     <inertial>
       <origin xyz="-0.000176 0.010059 -0.024478" rpy="0 0 0"/>
-      <mass value="0.550811"/>
+      <mass value="0.096623"/>
       <inertia
         ixx="0.00109482916"
@@ -284,5 +284,5 @@
     <inertial>
       <origin xyz="-0.000176 0.010059 -0.024478" rpy="0 0 0"/>
-      <mass value="0.550811"/>
+      <mass value="0.096623"/>
       <inertia
         ixx="0.00109482916"
@@ -629,3 +629,25 @@
     </plugin>
   </gazebo>
+  <gazebo reference="camera_link">
+    <sensor name="camera" type="camera">
+      <pose> 0 0 0.25 0 0.7 1</pose>
+      <visualize>true</visualize>
+      <update_rate>10.0</update_rate>
+      <camera>
+        <horizontal_fov>1.0</horizontal_fov>
+        <image>
+          <format>R8G8B8</format>
+          <width>640</width>
+          <height>480</height>
+        </image>
+        <clip>
+          <near>0.05</near>
+          <far>1.0</far>
+        </clip>
+      </camera>
+      <plugin name="camera_controller" filename="libgazebo_ros_camera.so">
+        <frame_name>camera_optical_link</frame_name>
+      </plugin>
+    </sensor>
+  </gazebo>
 </robot>

Commit message: added sim camera, fixed some bugs and edited some files.

File: src/pavlov_description/urdf/pavlov_mini.urdf.xacro (robot description, xacro)
@@ -2,4 +2,6 @@
 <robot name="pavlov_mini" xmlns:xacro="http://ros.org/wiki/xacro">
   <xacro:arg name="is_ignition" default="true"/>
+  <!-- Simulation-only tweak: tilt camera down/up (radians). Negative looks down. -->
+  <xacro:arg name="camera_sensor_pitch" default="-0.15"/>
   <xacro:include filename="$(find pavlov_description)/urdf/pavlov_mini_ros2_control.xacro" />
   <link name="base_link">
@@ -27,24 +29,34 @@
     </collision>
   </link>
-  <link name="lidar_link">
-    <visual>
-      <geometry>
-        <mesh filename= "package://pavlov_description/meshes/lidar.dae"/>
-      </geometry>
-    </visual>
-    <inertial>
-      <origin xyz="0.000 0.000 0.000" rpy ="0.000 0.000 0.000"/>
+  <link name="camera_link">
+    <visual>
+      <origin xyz="0.0 0.0 0.0" rpy="0.0 0.0 0.0"/>
+      <geometry>
+        <box size="0.030 0.030 0.030"/>
+      </geometry>
+      <material name="black">
+        <color rgba="0.1 0.1 0.1 1.0"/>
+      </material>
+    </visual>
+    <inertial>
       <mass value="0.050"/>
-      <inertia
-        ixx="0.00092" ixy="0.00000" ixz="0.00001"
-        iyy="0.00094" iyz="0.00000"
-        izz="0.00093"/>
-    </inertial>
-    <collision>
-      <origin xyz="0.010 0.000 -0.015" rpy ="0.000 0.000 0.000"/>
-      <geometry>
-        <box size="0.080 0.060 0.050"/>
-      </geometry>
-    </collision>
+      <inertia ixx="0.000001" ixy="0.0" ixz="0.0"
+              iyy="0.000001" iyz="0.0"
+              izz="0.000001"/>
+    </inertial>
+    <collision>
+      <origin xyz="0.0 0.0 0.0" rpy="0.0 0.0 0.0"/>
+      <geometry>
+        <box size="0.030 0.030 0.030"/>
+      </geometry>
+    </collision>
+  </link>
+  <link name="camera_optical_frame">
+    <inertial>
+      <mass value="0.001"/>
+      <inertia ixx="0.000001" ixy="0.0" ixz="0.0"
+              iyy="0.000001" iyz="0.0"
+              izz="0.000001"/>
+    </inertial>
   </link>
   <link name="hip_fl_ref">
@@ -493,8 +505,13 @@
   </link>
   <!-- JOINTS -->
-  <joint name="lidar" type="fixed" dont_collapse="true">
+  <joint name="camera_joint" type="fixed" dont_collapse="true">
     <parent link="base_link"/>
-    <child  link="lidar_link"/>
-    <origin xyz="0.04312 0.00000 0.08341"/>
+    <child link="camera_link"/>
+    <origin xyz="0.04312 0.00000 0.08341" rpy="0.0 0.0 0.0"/>
+  </joint>
+  <joint name="camera_optical_frame_joint" type="fixed" dont_collapse="true">
+    <parent link="camera_link"/>
+    <child link="camera_optical_frame"/>
+    <origin xyz="0.0 0.0 0.0" rpy="-1.5708 0.0 -1.5708"/>
   </joint>
   <joint name="fl_ref" type="fixed" dont_collapse="true">
@@ -629,3 +646,33 @@
     </plugin>
   </gazebo>
+  <!--
+    NOTE: Gazebo Sim's URDF->SDF conversion collapses fixed joints, so sensors end up
+    attached to the parent lumped link (typically `base_link`). To keep Gazebo topic
+    names predictable, attach the camera sensor to `base_link` with the full optical
+    pose.
+  -->
+  <gazebo reference="base_link">
+    <sensor name="camera_sensor" type="camera">
+      <!--
+        Gazebo camera looks along +X. Keep it aligned with base_link (+X forward),
+        and just tilt it in pitch so it can see the ground / target.
+      -->
+      <pose>0.04312 0 0.08341 0 $(arg camera_sensor_pitch) 0</pose>
+      <always_on>1</always_on>
+      <update_rate>30</update_rate>
+      <visualize>true</visualize>
+      <camera>
+        <horizontal_fov>1.3962634</horizontal_fov>
+        <image>
+          <width>640</width>
+          <height>480</height>
+          <format>R8G8B8</format>
+        </image>
+        <clip>
+          <near>0.02</near>
+          <far>10.0</far>
+        </clip>
+      </camera>
+    </sensor>
+  </gazebo>
 </robot>
